Commit message: added collision files

File: Humanoid_trial_v1/urdf/Humanoid_trial_v1.urdf (robot description, URDF)
Before this commit: robot Humanoid_trial_v1, 29 links, 28 joints
Links:
- link Head_Horizontal_Joint: geometry collision mesh filename=package://Humanoid_trial_v1/meshes/Head_Horizontal_Joint_co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; visual mesh filename=package://Humanoid_trial_v1/meshes/Head_Horizontal_Joint.STL
- link Head_Horizontal_Link: geometry collision mesh filename=package://Humanoid_trial_v1/meshes/Head_Horizontal_Link_col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; visual mesh filename=package://Humanoid_trial_v1/meshes/Head_Horizontal_Link.STL
- link Head_Vertical_Joint: geometry collision mesh filename=package://Humanoid_trial_v1/meshes/Head_Vertical_Joint_col.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; visual mesh filename=package://Humanoid_trial_v1/meshes/Head_Vertical_Joint.STL
- link Head_Vertical_Link: geometry collision mesh filename=package://Humanoid_trial_v1/meshes/Head_Vertical_Link_col.S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; visual mesh filename=package://Humanoid_trial_v1/meshes/Head_Vertical_Link.STL
- link Left_Calf_Joint: geometry collision mesh filename=package://Humanoid_trial_v1/meshes/Left_Calf_Joint_col.STL; visual mesh filename=package://Humanoid_trial_v1/meshes/Left_Calf_Joint.STL
- link Left_Calf_Link: geometry collision mesh filename=package://Humanoid_trial_v1/meshes/Left_Calf_Link_col.STL; visual mesh filename=package://Humanoid_trial_v1/meshes/Left_Calf_Link.STL
- link Left_Foot_Link: geometry collision mesh filename=package://Humanoid_trial_v1/meshes/Left_Foot_Link_col.STL; visual mesh filename=package://Humanoid_trial_v1/meshes/Left_Foot_Link.STL
- link Left_Hip_Joint: geometry collision mesh filename=package://Humanoid_trial_v1/meshes/Left_Hip_Joint_col.STL; visual mesh filename=package://Humanoid_trial_v1/meshes/Left_Hip_Joint.STL
- link Left_Rot_Hip_Link: geometry collision mesh filename=package://Humanoid_trial_v1/meshes/Left_Rot_Hip_Link_col.STL; visual mesh filename=package://Humanoid_trial_v1/meshes/Left_Rot_Hip_Link.STL
- link Left_Thigh_Joint: geometry collision mesh filename=package://Humanoid_trial_v1/meshes/Left_Thigh_Joint_col.STL; visual mesh filename=package://Humanoid_trial_v1/meshes/Left_Thigh_Joint.STL
- link Left_Thigh_Link: geometry collision mesh filename=package://Humanoid_trial_v1/meshes/Left_Thigh_Link_col.STL; visual mesh filename=package://Humanoid_trial_v1/meshes/Left_Thigh_Link.STL
- link Right_Calf_Joint: geometry collision mesh filename=package://Humanoid_trial_v1/meshes/Right_Calf_Joint_col.STL; visual mesh filename=package://Humanoid_trial_v1/meshes/Right_Calf_Joint.STL
- link Right_Calf_Link: geometry collision mesh filename=package://Humanoid_trial_v1/meshes/Right_Calf_Link_col.STL; visual mesh filename=package://Humanoid_trial_v1/meshes/Right_Calf_Link.STL
- link Right_Foot_Link: geometry collision mesh filename=package://Humanoid_trial_v1/meshes/Right_Foot_Link_col.STL; visual mesh filename=package://Humanoid_trial_v1/meshes/Right_Foot_Link.STL
- link Right_Hip_Joint: geometry collision mesh filename=package://Humanoid_trial_v1/meshes/Right_Hip_Joint_col.STL; visual mesh filename=package://Humanoid_trial_v1/meshes/Right_Hip_Joint.STL
- link Right_Rot_Hip_Link: geometry collision mesh filename=package://Humanoid_trial_v1/meshes/Right_Rot_Hip_Link_col.S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; visual mesh filename=package://Humanoid_trial_v1/meshes/Right_Rot_Hip_Link.STL
- link Right_Thigh_Joint: geometry collision mesh filename=package://Humanoid_trial_v1/meshes/Right_Thigh_Joint_col.STL; visual mesh filename=package://Humanoid_trial_v1/meshes/Right_Thigh_Joint.STL
- link Right_Thigh_Link: geometry collision mesh filename=package://Humanoid_trial_v1/meshes/Right_Thigh_Link_col.STL; visual mesh filename=package://Humanoid_trial_v1/meshes/Right_Thigh_Link.STL
- link base_link: geometry collision mesh filename=package://Humanoid_trial_v1/meshes/base_link_col.STL; visual mesh filename=package://Humanoid_trial_v1/meshes/base_link.STL
