Commit message: added the files

File: humanoid_descripition/urdf/humanoid (copy).urdf (robot description, URDF)
Before this commit: robot humanoid, 18 links, 17 joints
Links:
- removed link camera_link
- added link Camera_Link, mass 0; visual mesh filename=package://humanoid_descripition/meshes/Camera.STL
- added link IMU_Link, mass 0.000704900526624758; collision mesh filename=package://humanoid_descripition/meshes/IMU.STL; visual mesh filename=package://humanoid_descripition/meshes/IMU.STL
- added link Lens_Link, mass 0
Joints:
- removed joint camera_joint
- added joint Camera_Joint: type fixed, parent Head_Vertical_Link, child Camera_Link, origin xyz=0 0 0 rpy=0 0 0
- added joint IMU_Joint: type fixed, parent Head_Horizontal_Link, child IMU_Link, origin xyz=0.00022338 0.00015602 0.0 rpy=0 0 0, axis 0 0 0
- added joint Lens_joint: type fixed, parent Head_Vertical_Link, child Lens_Link, origin xyz=-0.0249627342624163 0.0274630025807885 0.000388603128653991 rpy=-3.14159265358979 -0.0155915295359344 -3.14010933670462, axis 0 0 0

File: humanoid_descripition/urdf/humanoid_main.urdf (robot description, URDF)
Before this commit: robot humanoid, 18 links, 17 joints
Links:
- removed link camera_link
- added link Camera_Link, mass 0; visual mesh filename=package://humanoid_descripition/meshes/Camera.STL
- added link IMU_Link, mass 0.000704900526624758; collision mesh filename=package://humanoid_descripition/meshes/IMU.STL; visual mesh filename=package://humanoid_descripition/meshes/IMU.STL
- added link Lens_Link, mass 0
Joints:
- removed joint Camera
- added joint Camera_Joint: type fixed, parent Head_Vertical_Link, child Camera_Link, origin xyz=0 0 0 rpy=0 0 0
- added joint IMU_Joint: type fixed, parent Head_Horizontal_Link, child IMU_Link, origin xyz=0.00022338 0.00015602 0.0 rpy=0 0 0, axis 0 0 0
- added joint Lens_joint: type fixed, parent Head_Vertical_Link, child Lens_Link, origin xyz=-0.0249627342624163 0.0274630025807885 0.000388603128653991 rpy=-3.14159265358979 -0.0155915295359344 -3.14010933670462, axis 0 0 0
