Commit message: changed tged the axis

File: humanoid_descripition/urdf/humanoid.urdf (robot description, URDF)
Before this commit: robot humanoid, 17 links, 16 joints
Joints:
- joint Left_Calf_Joint: axis 0 0 0 -> 0 1 0
- joint Left_Hip_Joint: axis 0 1 0 -> 0 0 1
- joint Right_Thigh_Joint: axis 0 0 0 -> 0 1 0

Commit message: added IMU

File: humanoid_descripition/urdf/humanoid.urdf (robot description, URDF)
Before this commit: robot humanoid, 17 links, 16 joints
Links:
- added link imu_link
Joints:
- added joint imu_fixed: type fixed, parent Head_Horizontal_Link, child imu_link, origin xyz=0.0299 0 0.5242 rpy=0 0 0

Commit message: added imu plugins

File: humanoid_descripition/urdf/humanoid.urdf (robot description, URDF)
Before this commit: robot humanoid, 18 links, 17 joints
Links:
- removed link imu_link
- added link Camera_Link, mass 0; visual mesh filename=package://humanoid_descripition/meshes/Camera.STL
- added link IMU_Link, mass 0.000704900526624758; collision mesh filename=package://humanoid_descripition/meshes/IMU.STL; visual mesh filename=package://humanoid_descripition/meshes/IMU.STL
- added link Lens_Link, mass 0
- link base_link: mass 1.51039036009517 -> 1.5156152965091
Joints:
- removed joint imu_fixed
- added joint Camera_Joint: type fixed, parent Head_Vertical_Link, child Camera_Link, origin xyz=0 0 0 rpy=0 0 0
- added joint IMU_Joint: type fixed, parent Head_Horizontal_Link, child IMU_Link, origin xyz=0.00022338 0.00015602 0.0 rpy=0 0 0, axis 0 0 0
- added joint Lens_joint: type fixed, parent Head_Vertical_Link, child Lens_Link, origin xyz=-0.0249627342624163 0.0274630025807885 0.000388603128653991 rpy=-3.14159265358979 -0.0155915295359344 -3.14010933670462, axis 0 0 0

Commit message: added t7nyka

File: humanoid_descripition/urdf/humanoid.urdf (robot description, URDF)
Before this commit: robot humanoid, 20 links, 19 joints
Links:
- added link base_footprint
Joints:
- added joint base_fixed: type fixed, parent base_footprint, child base_link, origin xyz=0 0 0 rpy=0 0 0

Commit message: Added a Vector of Chains to store the chain of each segement

File: humanoid_descripition/urdf/humanoid.urdf (robot description, URDF)
Before this commit: robot humanoid, 21 links, 20 joints
Links:
- removed link Left_Lower_Shoulder Link
- removed link base_footprint
- added link Left_Lower_Shoulder_Link, mass 0.116130359952787; collision mesh filename=package://humanoid_descripition/meshes/Left_Lower_Shoulder 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; visual mesh filename=package://humanoid_descripition/meshes/Left_Lower_Shoulder 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
- added link dummy
Joints:
- removed joint base_fixed
- added joint dummy_joint: type fixed, parent dummy, child base_link
- joint Left_Lower_Shoulder_Joint: child Left_Lower_Shoulder Link -> Left_Lower_Shoulder_Link

Commit message: set foot as fixed in urdf and modified c++ file

File: humanoid_descripition/urdf/humanoid.urdf (robot description, URDF)
Before this commit: robot humanoid, 21 links, 20 joints
Joints:
- joint Left_foot_Joint: type revolute -> fixed
- joint Right_Foot_Joint: type revolute -> fixed

Commit message: modified foot controller

File: humanoid_descripition/urdf/humanoid.urdf (robot description, URDF)
Before this commit: robot humanoid, 21 links, 20 joints
Joints:
- joint Left_foot_Joint: type fixed -> revolute
- joint Right_Foot_Joint: type fixed -> revolute

Commit message: modified the leg stl and urdf

File: humanoid_descripition/urdf/humanoid.urdf (robot description, URDF)
Before this commit: robot humanoid, 21 links, 20 joints
Links:
- link Left_foot_Link: mass 0.22826527251043 -> 0.228574752469723
- link Right_Foot_Link: mass 0.228265252831077 -> 0.228574752469723

Commit message: midified el the values of pid in control.yamel and changed joints axis in urdf

File: humanoid_descripition/urdf/humanoid.urdf (robot description, URDF)
Before this commit: robot humanoid, 21 links, 20 joints
Joints:
- joint Head_Horizontal_Joint: limit lower=-3.14 upper=3.14 effort=1.078 velocity=6.159 -> lower=-3.14 upper=3.14 effort=6 velocity=6.159
- joint Right_Calf_Joint: axis 0 -1 0 -> 0 1 0
